Commit message: feat(control): Implement Module 3 ros2_control integration

File: src/mower_description/urdf/mower.urdf.xacro (robot description, xacro)
@@ -1,316 +1,25 @@
 <?xml version="1.0"?>
 <robot xmlns:xacro="http://www.ros.org/wiki/xacro" name="mower">
-  <!-- Include materials -->
-  <material name="blue">
-    <color rgba="0.0 0.0 0.8 1.0"/>
-  </material>
-  <material name="red">
-    <color rgba="0.8 0.0 0.0 1.0"/>
-  </material>
-  <material name="green">
-    <color rgba="0.0 0.8 0.0 1.0"/>
-  </material>
-  <material name="grey">
-    <color rgba="0.5 0.5 0.5 1.0"/>
-  </material>
-  <material name="black">
-    <color rgba="0.0 0.0 0.0 1.0"/>
-  </material>
-  <!-- Base link - central reference frame -->
-  <link name="base_link">
-    <!-- This is just a reference frame, no visual or collision geometry -->
-  </link>
-  <!-- Chassis link - main body of the robot -->
-  <link name="chassis">
-    <visual>
-      <geometry>
-        <!-- Chassis dimensions: L:19cm, W:44cm, H:22cm -->
-        <box size="0.19 0.44 0.22"/>
-      </geometry>
-      <material name="blue"/>
-    </visual>
-    <collision>
-      <geometry>
-        <box size="0.19 0.44 0.22"/>
-      </geometry>
-    </collision>
-    <inertial>
-      <mass value="2.27"/>
-      <origin xyz="0 0 0" rpy="0 0 0"/>
-      <!-- Box inertia: m/12 * [y²+z², x²+z², x²+y²] -->
-      <!-- x=0.19, y=0.44, z=0.22 -->
-      <!-- Ixx = 2.27/12 * (0.44² + 0.22²) = 0.189 * (0.1936 + 0.0484) = 0.0457 -->
-      <!-- Iyy = 2.27/12 * (0.19² + 0.22²) = 0.189 * (0.0361 + 0.0484) = 0.0160 -->
-      <!-- Izz = 2.27/12 * (0.19² + 0.44²) = 0.189 * (0.0361 + 0.1936) = 0.0434 -->
-      <inertia ixx="0.0457" ixy="0.0" ixz="0.0"
-               iyy="0.0160" iyz="0.0"
-               izz="0.0434"/>
-    </inertial>
-  </link>
-  <!-- Joint connecting chassis to base_link -->
-  <joint name="chassis_joint" type="fixed">
-    <parent link="base_link"/>
-    <child link="chassis"/>
-    <!-- Position chassis so its bottom is at wheel center height (9.75cm)
-         Chassis height is 22cm, so center should be at 9.75 + 11 = 20.75cm -->
-    <origin xyz="0.0 0.0 0.2075" rpy="0 0 0"/>
-  </joint>
-  <!-- Left Drive Wheel -->
-  <link name="left_wheel">
-    <visual>
-      <geometry>
-        <!-- Wheel dimensions: Ø19.5cm, W:3.6cm -->
-        <cylinder radius="0.0975" length="0.036"/>
-      </geometry>
-      <material name="black"/>
-    </visual>
-    <collision>
-      <geometry>
-        <cylinder radius="0.0975" length="0.036"/>
-      </geometry>
-    </collision>
-    <inertial>
-      <mass value="1.81"/>
-      <origin xyz="0 0 0" rpy="0 0 0"/>
-      <!-- Cylinder inertia: m/12 * [3r²+l², 3r²+l², 6r²] -->
-      <!-- r=0.0975, l=0.036 -->
-      <!-- Ixx = 1.81/12 * (3*0.0975² + 0.036²) = 0.151 * (0.02847 + 0.001296) = 0.00449 -->
-      <!-- Iyy = 1.81/12 * (3*0.0975² + 0.036²) = 0.151 * (0.02847 + 0.001296) = 0.00449 -->
-      <!-- Izz = 1.81/12 * (6*0.0975²) = 0.151 * 0.05693 = 0.00860 -->
-      <inertia ixx="0.00449" ixy="0.0" ixz="0.0"
-               iyy="0.00449" iyz="0.0"
-               izz="0.00860"/>
-    </inertial>
-  </link>
-  <!-- Left wheel joint -->
-  <joint name="left_wheel_joint" type="continuous">
-    <parent link="base_link"/>
-    <child link="left_wheel"/>
-    <!-- Position: At (0, 23cm, 9.75cm) -->
-    <origin xyz="0.0 0.23 0.0975" rpy="-1.5707963 0 0"/>
-    <axis xyz="0 0 1"/>
-  </joint>
-  <!-- Right Drive Wheel -->
-  <link name="right_wheel">
-    <visual>
-      <geometry>
-        <!-- Wheel dimensions: Ø19.5cm, W:3.6cm -->
-        <cylinder radius="0.0975" length="0.036"/>
-      </geometry>
-      <material name="black"/>
-    </visual>
-    <collision>
-      <geometry>
-        <cylinder radius="0.0975" length="0.036"/>
-      </geometry>
-    </collision>
-    <inertial>
-      <mass value="1.81"/>
-      <origin xyz="0 0 0" rpy="0 0 0"/>
-      <!-- Cylinder inertia: m/12 * [3r²+l², 3r²+l², 6r²] -->
-      <!-- r=0.0975, l=0.036 -->
-      <!-- Ixx = 1.81/12 * (3*0.0975² + 0.036²) = 0.151 * (0.02847 + 0.001296) = 0.00449 -->
-      <!-- Iyy = 1.81/12 * (3*0.0975² + 0.036²) = 0.151 * (0.02847 + 0.001296) = 0.00449 -->
-      <!-- Izz = 1.81/12 * (6*0.0975²) = 0.151 * 0.05693 = 0.00860 -->
-      <inertia ixx="0.00449" ixy="0.0" ixz="0.0"
-               iyy="0.00449" iyz="0.0"
-               izz="0.00860"/>
-    </inertial>
-  </link>
-  <!-- Right wheel joint -->
-  <joint name="right_wheel_joint" type="continuous">
-    <parent link="base_link"/>
-    <child link="right_wheel"/>
-    <!-- Position: At (0, -23cm, 9.75cm) -->
-    <origin xyz="0.0 -0.23 0.0975" rpy="1.5707963 0 0"/>
-    <axis xyz="0 0 1"/>
-  </joint>
-  <!-- Counterweight -->
-  <link name="counterweight">
-    <visual>
-      <geometry>
-        <!-- Counterweight dimensions: L:21cm, W:13cm, H:13cm -->
-        <box size="0.21 0.13 0.13"/>
-      </geometry>
-      <material name="grey"/>
-    </visual>
-    <collision>
-      <geometry>
-        <box size="0.21 0.13 0.13"/>
-      </geometry>
-    </collision>
-    <inertial>
-      <mass value="9.07"/>
-      <origin xyz="0 0 0" rpy="0 0 0"/>
-      <!-- Box inertia: m/12 * [y²+z², x²+z², x²+y²] -->
-      <!-- x=0.21, y=0.13, z=0.13 -->
-      <!-- Ixx = 9.07/12 * (0.13² + 0.13²) = 0.756 * (0.0169 + 0.0169) = 0.0255 -->
-      <!-- Iyy = 9.07/12 * (0.21² + 0.13²) = 0.756 * (0.0441 + 0.0169) = 0.0461 -->
-      <!-- Izz = 9.07/12 * (0.21² + 0.13²) = 0.756 * (0.0441 + 0.0169) = 0.0461 -->
-      <inertia ixx="0.0255" ixy="0.0" ixz="0.0"
-               iyy="0.0461" iyz="0.0"
-               izz="0.0461"/>
-    </inertial>
-  </link>
-  <!-- Counterweight joint - fixed to chassis -->
-  <joint name="counterweight_joint" type="fixed">
-    <parent link="chassis"/>
-    <child link="counterweight"/>
-    <!-- Position at rear of chassis, butting up against it
-         Chassis length is 19cm, so half is 9.5cm
-         Counterweight length is 21cm, so half is 10.5cm
-         Total distance from chassis center to counterweight center: 9.5/2 + 10.5 = 20cm
-         Counterweight bottom should align with chassis bottom:
-         Chassis center at 20.75cm, counterweight height 13cm
-         Counterweight center should be at 9.75 + 6.5 = 16.25cm
-         Relative to chassis: 16.25 - 20.75 = -4.5cm -->
-    <origin xyz="-0.20 0.0 -0.045" rpy="0 0 0"/>
-  </joint>
-  <!-- Front Roller -->
-  <link name="front_roller">
-    <visual>
-      <geometry>
-        <!-- Front roller dimensions: Ø8.89cm, W:33cm -->
-        <cylinder radius="0.04445" length="0.33"/>
-      </geometry>
-      <material name="green"/>
-    </visual>
-    <collision>
-      <geometry>
-        <cylinder radius="0.04445" length="0.33"/>
-      </geometry>
-    </collision>
-    <inertial>
-      <mass value="0.45"/>
-      <origin xyz="0 0 0" rpy="0 0 0"/>
-      <!-- Cylinder inertia: m/12 * [3r²+l², 3r²+l², 6r²] -->
-      <!-- r=0.04445, l=0.33 -->
-      <!-- Ixx = 0.45/12 * (3*0.04445² + 0.33²) = 0.0375 * (0.00593 + 0.1089) = 0.00431 -->
-      <!-- Iyy = 0.45/12 * (3*0.04445² + 0.33²) = 0.0375 * (0.00593 + 0.1089) = 0.00431 -->
-      <!-- Izz = 0.45/12 * (6*0.04445²) = 0.0375 * 0.01185 = 0.000444 -->
-      <inertia ixx="0.00431" ixy="0.0" ixz="0.0"
-               iyy="0.00431" iyz="0.0"
-               izz="0.000444"/>
-    </inertial>
-  </link>
-  <!-- Front roller joint -->
-  <joint name="front_roller_joint" type="continuous">
-    <parent link="base_link"/>
-    <child link="front_roller"/>
-    <!-- Position: At (48cm, 0, 4.445cm) -->
-    <origin xyz="0.48 0.0 0.04445" rpy="-1.5707963 0 0"/>
-    <axis xyz="0 0 1"/>
-  </joint>
-  <!-- Cutting Reel -->
-  <link name="reel">
-    <visual>
-      <geometry>
-        <!-- Reel dimensions: Ø17.5cm, W:47cm -->
-        <cylinder radius="0.0875" length="0.47"/>
-      </geometry>
-      <material name="red"/>
-    </visual>
-    <collision>
-      <geometry>
-        <cylinder radius="0.0875" length="0.47"/>
-      </geometry>
-    </collision>
-    <inertial>
-      <mass value="11.34"/>
-      <origin xyz="0 0 0" rpy="0 0 0"/>
-      <!-- Cylinder inertia: m/12 * [3r²+l², 3r²+l², 6r²] -->
-      <!-- r=0.0875, l=0.47 -->
-      <!-- Ixx = 11.34/12 * (3*0.0875² + 0.47²) = 0.945 * (0.0229 + 0.2209) = 0.230 -->
-      <!-- Iyy = 11.34/12 * (3*0.0875² + 0.47²) = 0.945 * (0.0229 + 0.2209) = 0.230 -->
-      <!-- Izz = 11.34/12 * (6*0.0875²) = 0.945 * 0.0459 = 0.0434 -->
-      <inertia ixx="0.230" ixy="0.0" ixz="0.0"
-               iyy="0.230" iyz="0.0"
-               izz="0.0434"/>
-    </inertial>
-  </link>
-  <!-- Reel joint -->
-  <joint name="reel_joint" type="continuous">
-    <parent link="base_link"/>
-    <child link="reel"/>
-    <!-- Position: Raise reel 3cm off ground
-         Reel radius is 8.75cm, so center should be at 3 + 8.75 = 11.75cm -->
-    <origin xyz="0.30 0.0 0.1175" rpy="-1.5707963 0 0"/>
-    <axis xyz="0 0 1"/>
-  </joint>
-  <!-- Reel Motor -->
-  <link name="reel_motor">
-    <visual>
-      <geometry>
-        <!-- Motor dimensions: cylinder with 2cm radius, 12cm height -->
-        <cylinder radius="0.02" length="0.12"/>
-      </geometry>
-      <material name="black"/>
-    </visual>
-    <collision>
-      <geometry>
-        <cylinder radius="0.02" length="0.12"/>
-      </geometry>
-    </collision>
-    <inertial>
-      <mass value="1.0"/>
-      <origin xyz="0 0 0" rpy="0 0 0"/>
-      <!-- Cylinder inertia: m/12 * [3r²+l², 3r²+l², 6r²] -->
-      <!-- r=0.02, l=0.12 -->
-      <!-- Ixx = 1.0/12 * (3*0.02² + 0.12²) = 0.0833 * (0.0012 + 0.0144) = 0.00130 -->
-      <!-- Iyy = 1.0/12 * (3*0.02² + 0.12²) = 0.0833 * (0.0012 + 0.0144) = 0.00130 -->
-      <!-- Izz = 1.0/12 * (6*0.02²) = 0.0833 * 0.0024 = 0.000200 -->
-      <inertia ixx="0.00130" ixy="0.0" ixz="0.0"
-               iyy="0.00130" iyz="0.0"
-               izz="0.000200"/>
-    </inertial>
-  </link>
-  <!-- Reel motor joint - fixed to chassis -->
-  <joint name="reel_motor_joint" type="fixed">
-    <parent link="chassis"/>
-    <child link="reel_motor"/>
-    <!-- Position: At (21.8cm, -23.5cm, 17.55cm) relative to base_link
-         Since chassis is now at Z=20.75cm, adjust relative position:
-         Z_relative = 17.55 - 20.75 = -3.2cm -->
-    <origin xyz="0.218 -0.235 -0.032" rpy="-1.5707963 0 0"/>
-  </joint>
-  <!-- ROS2 Control Integration -->
-  <ros2_control name="GazeboSystem" type="system">
-    <hardware>
-      <plugin>gz_ros2_control/GazeboSystem</plugin>
-    </hardware>
-    <!-- Left Wheel Joint Control -->
-    <joint name="left_wheel_joint">
-      <command_interface name="velocity">
-        <param name="min">-10</param>
-        <param name="max">10</param>
-      </command_interface>
-      <state_interface name="position"/>
-      <state_interface name="velocity"/>
-    </joint>
-    <!-- Right Wheel Joint Control -->
-    <joint name="right_wheel_joint">
-      <command_interface name="velocity">
-        <param name="min">-10</param>
-        <param name="max">10</param>
-      </command_interface>
-      <state_interface name="position"/>
-      <state_interface name="velocity"/>
-    </joint>
-    <!-- Reel Joint Control -->
-    <joint name="reel_joint">
-      <command_interface name="velocity">
-        <param name="min">-20</param>
-        <param name="max">20</param>
-      </command_interface>
-      <state_interface name="position"/>
-      <state_interface name="velocity"/>
-    </joint>
-  </ros2_control>
-  <!-- Gazebo ROS2 Control Plugin -->
-  <gazebo>
-    <plugin filename="gz_ros2_control-system" name="gz_ros2_control::GazeboSimROS2ControlPlugin">
-      <parameters>/home/tyler/mower_ws/install/mower_control/share/mower_control/config/mower_controllers.yaml</parameters>
-    </plugin>
-  </gazebo>
+  <!--
+    Autonomous Mower Robot Description - Main Assembly File
+    This is the main URDF/XACRO file that assembles the complete mower robot
+    from modular component files. This modular approach provides:
+    - Better maintainability: Each component can be modified independently
+    - Improved reusability: Components can be reused in different configurations
+    - Enhanced clarity: Logical separation makes the model easier to understand
+    - Better collaboration: Multiple developers can work on different components
+    - Easy customization: Components can be easily swapped or modified
+    Component Structure:
+    - materials.xacro: Material definitions and colors
+    - chassis.xacro: Main body structure and counterweight
+    - wheels.xacro: Drive wheels and their joints
+    - cutting_system.xacro: Reel, front roller, and motor components
+    - ros2_control.xacro: Control interfaces for simulation and hardware
+  -->
+  <!-- Include all component files -->
+  <xacro:include filename="$(find mower_description)/urdf/components/materials.xacro"/>
+  <xacro:include filename="$(find mower_description)/urdf/components/chassis.xacro"/>
+  <xacro:include filename="$(find mower_description)/urdf/components/wheels.xacro"/>
+  <xacro:include filename="$(find mower_description)/urdf/components/cutting_system.xacro"/>
+  <xacro:include filename="$(find mower_description)/urdf/components/ros2_control.xacro"/>
 </robot>
-```
