Commit message: fix(control): Resolve clock synchronization and complete Module 3

File: src/mower_description/urdf/components/cutting_system.xacro (robot description, xacro)
@@ -90,5 +90,5 @@
       <inertia ixx="${reel_motor_mass * (0.05*0.05 + 0.05*0.05) / 12}"
                ixy="0.0" ixz="0.0"
-               iyy="-${reel_motor_mass * (0.05*0.05 + 0.05*0.05) / 12}"
+               iyy="${reel_motor_mass * (0.05*0.05 + 0.05*0.05) / 12}"
                iyz="0.0"
                izz="${reel_motor_mass * (0.05*0.05 + 0.05*0.05) / 12}"/>

File: src/mower_description/urdf/components/sensors.xacro (robot description, xacro)
@@ -30,5 +30,5 @@
     <parent link="base_link"/>
     <child link="imu_link"/>
-    <origin xyz="${imu_x} ${imu_y} ${imu_z - wheel_radius - chassis_height/2}" rpy="0 0 0"/>
+    <origin xyz="${imu_x} ${imu_y} ${imu_z - wheel_radius}" rpy="0 0 0"/>
   </joint>
   <!-- GPS Sensor Link -->
@@ -36,5 +36,5 @@
     <visual>
       <geometry>
-        <box size="0.03 0.03 0.01"/>
+        <box size="0.03 0.03 0.04"/>
       </geometry>
       <material name="orange"/>
@@ -42,5 +42,5 @@
     <collision>
       <geometry>
-        <box size="0.03 0.03 0.01"/>
+        <box size="0.03 0.03 0.04"/>
       </geometry>
     </collision>
@@ -54,5 +54,5 @@
     <parent link="base_link"/>
     <child link="gps_link"/>
-    <origin xyz="${gps_x} ${gps_y} ${gps_z - wheel_radius - chassis_height/2}" rpy="0 0 0"/>
+    <origin xyz="${gps_x} ${gps_y} ${gps_z - wheel_radius}" rpy="0 0 0"/>
   </joint>
 </robot>
