Commit message: feat: Complete Phase 1 foundation with modular URDF and ros2_control integration

File: src/mower_description/urdf/components/chassis.xacro (robot description, xacro)
@@ -4,88 +4,70 @@
     Chassis Component
     This file defines the main structural elements of the mower:
-    - base_link: Central reference frame at ground level
-    - chassis: Main body of the robot
+    - base_link: Main chassis body (following reference structure)
     - counterweight: Rear counterweight for balance
-    All dimensions and masses are based on the Product Requirements Document.
+    All dimensions and masses use properties from properties.xacro.
   -->
-  <!-- Base link - central reference frame at ground level -->
+  <!-- Root Link (dummy link without inertia for KDL compatibility) -->
+  <link name="base_footprint">
+    <!-- No inertia on root link - KDL requirement -->
+  </link>
+  <!-- Fixed joint connecting root to actual chassis -->
+  <joint name="base_footprint_joint" type="fixed">
+    <parent link="base_footprint"/>
+    <child link="base_link"/>
+    <origin xyz="0 0 ${wheel_radius}" rpy="0 0 0"/>
+  </joint>
+  <!-- Base Link (main chassis) - now as child link with inertia -->
   <link name="base_link">
-    <!-- This is just a reference frame, no visual or collision geometry -->
-  </link>
-  <!-- Chassis link - main body of the robot -->
-  <link name="chassis">
+    <inertial>
+      <origin xyz="0 0 0" rpy="0 0 0"/>
+      <mass value="${chassis_mass}"/>
+      <inertia ixx="${chassis_mass * (chassis_width*chassis_width + chassis_height*chassis_height) / 12}"
+               ixy="0.0" ixz="0.0"
+               iyy="${chassis_mass * (chassis_length*chassis_length + chassis_height*chassis_height) / 12}"
+               iyz="0.0"
+               izz="${chassis_mass * (chassis_length*chassis_length + chassis_width*chassis_width) / 12}"/>
+    </inertial>
     <visual>
+      <origin xyz="0 0 0" rpy="0 0 0"/>
       <geometry>
-        <!-- Chassis dimensions: L:19cm, W:44cm, H:22cm -->
-        <box size="0.19 0.44 0.22"/>
+        <box size="${chassis_length} ${chassis_width} ${chassis_height}"/>
       </geometry>
       <material name="blue"/>
     </visual>
     <collision>
+      <origin xyz="0 0 0" rpy="0 0 0"/>
       <geometry>
-        <box size="0.19 0.44 0.22"/>
+        <box size="${chassis_length} ${chassis_width} ${chassis_height}"/>
+      </geometry>
+    </collision>
+  </link>
+  <!-- Counterweight Link -->
+  <link name="counterweight">
+    <visual>
+      <geometry>
+        <box size="${counterweight_length} ${counterweight_width} ${counterweight_height}"/>
+      </geometry>
+      <material name="gray"/>
+    </visual>
+    <collision>
+      <geometry>
+        <box size="${counterweight_length} ${counterweight_width} ${counterweight_height}"/>
       </geometry>
     </collision>
     <inertial>
-      <mass value="2.27"/>
-      <origin xyz="0 0 0" rpy="0 0 0"/>
-      <!-- Box inertia: m/12 * [y²+z², x²+z², x²+y²] -->
-      <!-- x=0.19, y=0.44, z=0.22 -->
-      <!-- Ixx = 2.27/12 * (0.44² + 0.22²) = 0.189 * (0.1936 + 0.0484) = 0.0457 -->
-      <!-- Iyy = 2.27/12 * (0.19² + 0.22²) = 0.189 * (0.0361 + 0.0484) = 0.0160 -->
-      <!-- Izz = 2.27/12 * (0.19² + 0.44²) = 0.189 * (0.0361 + 0.1936) = 0.0434 -->
-      <inertia ixx="0.0457" ixy="0.0" ixz="0.0"
-               iyy="0.0160" iyz="0.0"
-               izz="0.0434"/>
+      <mass value="${counterweight_mass}"/>
+      <inertia ixx="${counterweight_mass * (counterweight_width*counterweight_width + counterweight_height*counterweight_height) / 12}"
+               ixy="0.0" ixz="0.0"
+               iyy="${counterweight_mass * (counterweight_length*counterweight_length + counterweight_height*counterweight_height) / 12}"
+               iyz="0.0"
+               izz="${counterweight_mass * (counterweight_length*counterweight_length + counterweight_width*counterweight_width) / 12}"/>
     </inertial>
   </link>
-  <!-- Joint connecting chassis to base_link -->
-  <joint name="chassis_joint" type="fixed">
+  <!-- Counterweight Joint -->
+  <joint name="chassis_to_counterweight" type="fixed">
     <parent link="base_link"/>
-    <child link="chassis"/>
-    <!-- Position chassis so its bottom is at wheel center height (9.75cm)
-         Chassis height is 22cm, so center should be at 9.75 + 11 = 20.75cm -->
-    <origin xyz="0.0 0.0 0.2075" rpy="0 0 0"/>
-  </joint>
-  <!-- Counterweight -->
-  <link name="counterweight">
-    <visual>
-      <geometry>
-        <!-- Counterweight dimensions: L:21cm, W:13cm, H:13cm -->
-        <box size="0.21 0.13 0.13"/>
-      </geometry>
-      <material name="grey"/>
-    </visual>
-    <collision>
-      <geometry>
-        <box size="0.21 0.13 0.13"/>
-      </geometry>
-    </collision>
-    <inertial>
-      <mass value="9.07"/>
-      <origin xyz="0 0 0" rpy="0 0 0"/>
-      <!-- Box inertia: m/12 * [y²+z², x²+z², x²+y²] -->
-      <!-- x=0.21, y=0.13, z=0.13 -->
-      <!-- Ixx = 9.07/12 * (0.13² + 0.13²) = 0.756 * (0.0169 + 0.0169) = 0.0255 -->
-      <!-- Iyy = 9.07/12 * (0.21² + 0.13²) = 0.756 * (0.0441 + 0.0169) = 0.0461 -->
-      <!-- Izz = 9.07/12 * (0.21² + 0.13²) = 0.756 * (0.0441 + 0.0169) = 0.0461 -->
-      <inertia ixx="0.0255" ixy="0.0" ixz="0.0"
-               iyy="0.0461" iyz="0.0"
-               izz="0.0461"/>
-    </inertial>
-  </link>
-  <!-- Counterweight joint - fixed to chassis -->
-  <joint name="counterweight_joint" type="fixed">
-    <parent link="chassis"/>
     <child link="counterweight"/>
-    <!-- Position at rear of chassis, butting up against it
-         Chassis length is 19cm, so half is 9.5cm
-         Counterweight length is 21cm, so half is 10.5cm
-         Total distance from chassis center to counterweight center: 9.5/2 + 10.5 = 20cm
-         Counterweight bottom should align with chassis bottom:
-         Chassis center at 20.75cm, counterweight height 13cm
-         Counterweight center should be at 9.75 + 6.5 = 16.25cm
-         Relative to chassis: 16.25 - 20.75 = -4.5cm -->
-    <origin xyz="-0.20 0.0 -0.045" rpy="0 0 0"/>
+    <origin xyz="-${(chassis_length + counterweight_length)/2} 0.0 -${(chassis_height - counterweight_height)/2}" rpy="0 0 0"/>
   </joint>
 </robot>

File: src/mower_description/urdf/components/cutting_system.xacro (robot description, xacro)
@@ -3,52 +3,79 @@
   <!--
     Cutting System Component
-    This file defines the cutting and support system of the mower:
+    This file defines the cutting and support system following the reference style:
     - front_roller: Front support roller
     - reel: Main cutting reel assembly
     - reel_motor: Motor that drives the cutting reel
-    The cutting system includes both active (reel) and passive (roller) elements.
-    Dimensions and masses are based on the Product Requirements Document.
+    All dimensions and masses use properties from properties.xacro.
   -->
-  <!-- Front Roller -->
+  <!-- Front Roller Link -->
   <link name="front_roller">
     <visual>
+      <origin xyz="0 0 0" rpy="${pi/2} 0 0"/>
       <geometry>
-        <!-- Front roller dimensions: Ø8.89cm, W:33cm -->
-        <cylinder radius="0.04445" length="0.33"/>
+        <cylinder radius="${front_roller_radius}" length="${front_roller_width}"/>
+      </geometry>
+      <material name="white"/>
+    </visual>
+    <collision>
+      <origin xyz="0 0 0" rpy="${pi/2} 0 0"/>
+      <geometry>
+        <cylinder radius="${front_roller_radius}" length="${front_roller_width}"/>
+      </geometry>
+    </collision>
+    <inertial>
+      <mass value="${front_roller_mass}"/>
+      <inertia ixx="${front_roller_mass * (3*front_roller_radius*front_roller_radius + front_roller_width*front_roller_width) / 12}"
+               ixy="0.0" ixz="0.0"
+               iyy="${front_roller_mass * front_roller_radius*front_roller_radius / 2}"
+               iyz="0.0"
+               izz="${front_roller_mass * (3*front_roller_radius*front_roller_radius + front_roller_width*front_roller_width) / 12}"/>
+    </inertial>
+  </link>
+  <!-- Front Roller Joint -->
+  <joint name="front_roller_joint" type="continuous">
+    <parent link="base_link"/>
+    <child link="front_roller"/>
+    <origin xyz="0.48 0.0 -${chassis_height/2 + front_roller_radius}" rpy="0 0 0"/>
+    <axis xyz="0 1 0"/>
+    <dynamics damping="0.5" friction="0.8"/>
+  </joint>
+  <!-- Reel Link -->
+  <link name="reel">
+    <visual>
+      <origin xyz="0 0 0" rpy="${pi/2} 0 0"/>
+      <geometry>
+        <cylinder radius="${reel_radius}" length="${reel_width}"/>
       </geometry>
       <material name="green"/>
     </visual>
     <collision>
+      <origin xyz="0 0 0" rpy="${pi/2} 0 0"/>
       <geometry>
-        <cylinder radius="0.04445" length="0.33"/>
+        <cylinder radius="${reel_radius}" length="${reel_width}"/>
       </geometry>
     </collision>
     <inertial>
-      <mass value="0.45"/>
-      <origin xyz="0 0 0" rpy="0 0 0"/>
-      <!-- Cylinder inertia: m/12 * [3r²+l², 3r²+l², 6r²] -->
-      <!-- r=0.04445, l=0.33 -->
-      <!-- Ixx = 0.45/12 * (3*0.04445² + 0.33²) = 0.0375 * (0.00593 + 0.1089) = 0.00431 -->
-      <!-- Iyy = 0.45/12 * (3*0.04445² + 0.33²) = 0.0375 * (0.00593 + 0.1089) = 0.00431 -->
-      <!-- Izz = 0.45/12 * (6*0.04445²) = 0.0375 * 0.01185 = 0.000444 -->
-      <inertia ixx="0.00431" ixy="0.0" ixz="0.0"
-               iyy="0.00431" iyz="0.0"
-               izz="0.000444"/>
+      <mass value="${reel_mass}"/>
+      <inertia ixx="${reel_mass * (3*reel_radius*reel_radius + reel_width*reel_width) / 12}"
+               ixy="0.0" ixz="0.0"
+               iyy="${reel_mass * reel_radius*reel_radius / 2}"
+               iyz="0.0"
+               izz="${reel_mass * (3*reel_radius*reel_radius + reel_width*reel_width) / 12}"/>
     </inertial>
   </link>
-  <!-- Front roller joint -->
-  <joint name="front_roller_joint" type="continuous">
+  <!-- Reel Joint -->
+  <joint name="reel_joint" type="continuous">
     <parent link="base_link"/>
-    <child link="front_roller"/>
-    <!-- Position: At (48cm, 0, 4.445cm) -->
-    <origin xyz="0.48 0.0 0.04445" rpy="-1.5707963 0 0"/>
-    <axis xyz="0 0 1"/>
+    <child link="reel"/>
+    <origin xyz="0.30 0.0 -${chassis_height/2 - 0.02}" rpy="0 0 0"/>
+    <axis xyz="0 1 0"/>
+    <dynamics damping="0.8" friction="1.2"/>
   </joint>
-  <!-- Cutting Reel -->
-  <link name="reel">
+  <!-- Reel Motor Link -->
+  <link name="reel_motor">
     <visual>
       <geometry>
-        <!-- Reel dimensions: Ø17.5cm, W:47cm -->
-        <cylinder radius="0.0875" length="0.47"/>
+        <box size="0.05 0.05 0.05"/>
       </geometry>
       <material name="red"/>
@@ -56,64 +83,21 @@
     <collision>
       <geometry>
-        <cylinder radius="0.0875" length="0.47"/>
+        <box size="0.05 0.05 0.05"/>
       </geometry>
     </collision>
     <inertial>
-      <mass value="11.34"/>
-      <origin xyz="0 0 0" rpy="0 0 0"/>
-      <!-- Cylinder inertia: m/12 * [3r²+l², 3r²+l², 6r²] -->
-      <!-- r=0.0875, l=0.47 -->
-      <!-- Ixx = 11.34/12 * (3*0.0875² + 0.47²) = 0.945 * (0.0229 + 0.2209) = 0.230 -->
-      <!-- Iyy = 11.34/12 * (3*0.0875² + 0.47²) = 0.945 * (0.0229 + 0.2209) = 0.230 -->
-      <!-- Izz = 11.34/12 * (6*0.0875²) = 0.945 * 0.0459 = 0.0434 -->
-      <inertia ixx="0.230" ixy="0.0" ixz="0.0"
-               iyy="0.230" iyz="0.0"
-               izz="0.0434"/>
+      <mass value="${reel_motor_mass}"/>
+      <inertia ixx="${reel_motor_mass * (0.05*0.05 + 0.05*0.05) / 12}"
+               ixy="0.0" ixz="0.0"
+               iyy="-${reel_motor_mass * (0.05*0.05 + 0.05*0.05) / 12}"
+               iyz="0.0"
+               izz="${reel_motor_mass * (0.05*0.05 + 0.05*0.05) / 12}"/>
     </inertial>
   </link>
-  <!-- Reel joint -->
-  <joint name="reel_joint" type="continuous">
+  <!-- Reel Motor Joint -->
+  <joint name="chassis_to_reel_motor" type="fixed">
     <parent link="base_link"/>
-    <child link="reel"/>
-    <!-- Position: Raise reel 3cm off ground
-         Reel radius is 8.75cm, so center should be at 3 + 8.75 = 11.75cm -->
-    <origin xyz="0.30 0.0 0.1175" rpy="-1.5707963 0 0"/>
-    <axis xyz="0 0 1"/>
-  </joint>
-  <!-- Reel Motor -->
-  <link name="reel_motor">
-    <visual>
-      <geometry>
-        <!-- Motor dimensions: cylinder with 2cm radius, 12cm height -->
-        <cylinder radius="0.02" length="0.12"/>
-      </geometry>
-      <material name="black"/>
-    </visual>
-    <collision>
-      <geometry>
-        <cylinder radius="0.02" length="0.12"/>
-      </geometry>
-    </collision>
-    <inertial>
-      <mass value="1.0"/>
-      <origin xyz="0 0 0" rpy="0 0 0"/>
-      <!-- Cylinder inertia: m/12 * [3r²+l², 3r²+l², 6r²] -->
-      <!-- r=0.02, l=0.12 -->
-      <!-- Ixx = 1.0/12 * (3*0.02² + 0.12²) = 0.0833 * (0.0012 + 0.0144) = 0.00130 -->
-      <!-- Iyy = 1.0/12 * (3*0.02² + 0.12²) = 0.0833 * (0.0012 + 0.0144) = 0.00130 -->
-      <!-- Izz = 1.0/12 * (6*0.02²) = 0.0833 * 0.0024 = 0.000200 -->
-      <inertia ixx="0.00130" ixy="0.0" ixz="0.0"
-               iyy="0.00130" iyz="0.0"
-               izz="0.000200"/>
-    </inertial>
-  </link>
-  <!-- Reel motor joint - fixed to chassis -->
-  <joint name="reel_motor_joint" type="fixed">
-    <parent link="chassis"/>
     <child link="reel_motor"/>
-    <!-- Position: At (21.8cm, -23.5cm, 17.55cm) relative to base_link
-         Since chassis is now at Z=20.75cm, adjust relative position:
-         Z_relative = 17.55 - 20.75 = -3.2cm -->
-    <origin xyz="0.218 -0.235 -0.032" rpy="-1.5707963 0 0"/>
+    <origin xyz="0.125 0.11 0.04" rpy="0 0 0"/>
   </joint>
 </robot>

File: src/mower_description/urdf/components/materials.xacro (robot description, xacro)
@@ -9,21 +9,33 @@
   <!-- Blue material for chassis -->
   <material name="blue">
-    <color rgba="0.0 0.0 0.8 1.0"/>
+    <color rgba="0.0 0.0 1.0 1.0"/>
   </material>
-  <!-- Red material for cutting reel -->
+  <!-- Red material for reel motor -->
   <material name="red">
-    <color rgba="0.8 0.0 0.0 1.0"/>
+    <color rgba="1.0 0.0 0.0 1.0"/>
   </material>
-  <!-- Green material for front roller -->
+  <!-- Green material for cutting reel -->
   <material name="green">
-    <color rgba="0.0 0.8 0.0 1.0"/>
+    <color rgba="0.0 1.0 0.0 1.0"/>
   </material>
-  <!-- Grey material for counterweight -->
-  <material name="grey">
+  <!-- Gray material for counterweight -->
+  <material name="gray">
     <color rgba="0.5 0.5 0.5 1.0"/>
   </material>
-  <!-- Black material for wheels and motor -->
+  <!-- Black material for wheels -->
   <material name="black">
     <color rgba="0.0 0.0 0.0 1.0"/>
   </material>
+  <!-- White material for front roller -->
+  <material name="white">
+    <color rgba="1.0 1.0 1.0 1.0"/>
+  </material>
+  <!-- Purple material for IMU -->
+  <material name="purple">
+    <color rgba="0.5 0.0 0.5 1.0"/>
+  </material>
+  <!-- Orange material for GPS -->
+  <material name="orange">
+    <color rgba="1.0 0.5 0.0 1.0"/>
+  </material>
 </robot>

File: src/mower_description/urdf/components/ros2_control.xacro (robot description, xacro)
@@ -12,40 +12,36 @@
   -->
   <!-- ROS2 Control Integration -->
-  <ros2_control name="GazeboSystem" type="system">
+  <ros2_control name="GazeboSimSystem" type="system">
     <hardware>
       <plugin>gz_ros2_control/GazeboSimSystem</plugin>
     </hardware>
-    <!-- Left Wheel Joint Control -->
-    <joint name="left_wheel_joint">
-      <command_interface name="velocity">
-        <param name="min">-10</param>
-        <param name="max">10</param>
-      </command_interface>
+    <!-- Right Wheel Joint -->
+    <joint name="right_wheel_joint">
+      <command_interface name="velocity"/>
       <state_interface name="position"/>
       <state_interface name="velocity"/>
     </joint>
-    <!-- Right Wheel Joint Control -->
-    <joint name="right_wheel_joint">
-      <command_interface name="velocity">
-        <param name="min">-10</param>
-        <param name="max">10</param>
-      </command_interface>
+    <!-- Left Wheel Joint -->
+    <joint name="left_wheel_joint">
+      <command_interface name="velocity"/>
       <state_interface name="position"/>
       <state_interface name="velocity"/>
     </joint>
-    <!-- Reel Joint Control -->
+    <!-- Reel Joint -->
     <joint name="reel_joint">
-      <command_interface name="velocity">
-        <param name="min">-20</param>
-        <param name="max">20</param>
-      </command_interface>
+      <command_interface name="velocity"/>
+      <state_interface name="position"/>
+      <state_interface name="velocity"/>
+    </joint>
+    <!-- Front Roller Joint (passive, state-only) -->
+    <joint name="front_roller_joint">
       <state_interface name="position"/>
       <state_interface name="velocity"/>
     </joint>
   </ros2_control>
-  <!-- Gazebo ROS2 Control Plugin -->
+  <!-- Gazebo ros2_control Plugin -->
   <gazebo>
-    <plugin filename="gz_ros2_control-system" name="gz_ros2_control::GazeboSimROS2ControlPlugin">
-      <parameters>/home/tyler/mower_ws/install/mower_control/share/mower_control/config/mower_controllers.yaml</parameters>
+    <plugin name="gz_ros2_control::GazeboSimROS2ControlPlugin" filename="libgz_ros2_control-system">
+      <parameters>$(find mower_control)/config/mower_controllers.yaml</parameters>
     </plugin>
   </gazebo>

File: src/mower_description/urdf/components/wheels.xacro (robot description, xacro)
@@ -3,80 +3,73 @@
   <!--
     Wheels Component
-    This file defines the drive wheels and their joints:
+    This file defines the drive wheels and their joints following the reference style:
+    - right_wheel: Right drive wheel with hub motor
     - left_wheel: Left drive wheel with hub motor
-    - right_wheel: Right drive wheel with hub motor
     - Continuous joints for wheel rotation
-    Both wheels are identical except for their position and rotation axis.
-    Dimensions and masses are based on the Product Requirements Document.
+    All dimensions and masses use properties from properties.xacro.
   -->
-  <!-- Left Drive Wheel -->
-  <link name="left_wheel">
+  <!-- Right Wheel Link -->
+  <link name="right_wheel">
     <visual>
+      <origin xyz="0 0 0" rpy="${pi/2} 0 0"/>
       <geometry>
-        <!-- Wheel dimensions: Ø19.5cm, W:3.6cm -->
-        <cylinder radius="0.0975" length="0.036"/>
+        <cylinder radius="${wheel_radius}" length="${wheel_width}"/>
       </geometry>
       <material name="black"/>
     </visual>
     <collision>
+      <origin xyz="0 0 0" rpy="${pi/2} 0 0"/>
       <geometry>
-        <cylinder radius="0.0975" length="0.036"/>
+        <cylinder radius="${wheel_radius}" length="${wheel_width}"/>
       </geometry>
     </collision>
     <inertial>
-      <mass value="1.81"/>
-      <origin xyz="0 0 0" rpy="0 0 0"/>
-      <!-- Cylinder inertia: m/12 * [3r²+l², 3r²+l², 6r²] -->
-      <!-- r=0.0975, l=0.036 -->
-      <!-- Ixx = 1.81/12 * (3*0.0975² + 0.036²) = 0.151 * (0.02847 + 0.001296) = 0.00449 -->
-      <!-- Iyy = 1.81/12 * (3*0.0975² + 0.036²) = 0.151 * (0.02847 + 0.001296) = 0.00449 -->
-      <!-- Izz = 1.81/12 * (6*0.0975²) = 0.151 * 0.05693 = 0.00860 -->
-      <inertia ixx="0.00449" ixy="0.0" ixz="0.0"
-               iyy="0.00449" iyz="0.0"
-               izz="0.00860"/>
+      <mass value="${wheel_mass}"/>
+      <inertia ixx="${wheel_mass * (3*wheel_radius*wheel_radius + wheel_width*wheel_width) / 12}"
+               ixy="0.0" ixz="0.0"
+               iyy="${wheel_mass * wheel_radius*wheel_radius / 2}"
+               iyz="0.0"
+               izz="${wheel_mass * (3*wheel_radius*wheel_radius + wheel_width*wheel_width) / 12}"/>
     </inertial>
   </link>
-  <!-- Left wheel joint -->
-  <joint name="left_wheel_joint" type="continuous">
+  <!-- Right Wheel Joint -->
+  <joint name="right_wheel_joint" type="continuous">
     <parent link="base_link"/>
-    <child link="left_wheel"/>
-    <!-- Position: At (0, 23cm, 9.75cm) -->
-    <origin xyz="0.0 0.23 0.0975" rpy="-1.5707963 0 0"/>
-    <axis xyz="0 0 1"/>
+    <child link="right_wheel"/>
+    <origin xyz="0.0 -${wheel_separation/2} -${chassis_height/2}" rpy="0 0 0"/>
+    <axis xyz="0 1 0"/>
+    <dynamics damping="0.7" friction="1.0"/>
   </joint>
-  <!-- Right Drive Wheel -->
-  <link name="right_wheel">
+  <!-- Left Wheel Link -->
+  <link name="left_wheel">
     <visual>
+      <origin xyz="0 0 0" rpy="${pi/2} 0 0"/>
       <geometry>
-        <!-- Wheel dimensions: Ø19.5cm, W:3.6cm -->
-        <cylinder radius="0.0975" length="0.036"/>
+        <cylinder radius="${wheel_radius}" length="${wheel_width}"/>
       </geometry>
       <material name="black"/>
     </visual>
     <collision>
+      <origin xyz="0 0 0" rpy="${pi/2} 0 0"/>
       <geometry>
-        <cylinder radius="0.0975" length="0.036"/>
+        <cylinder radius="${wheel_radius}" length="${wheel_width}"/>
       </geometry>
     </collision>
     <inertial>
-      <mass value="1.81"/>
-      <origin xyz="0 0 0" rpy="0 0 0"/>
-      <!-- Cylinder inertia: m/12 * [3r²+l², 3r²+l², 6r²] -->
-      <!-- r=0.0975, l=0.036 -->
-      <!-- Ixx = 1.81/12 * (3*0.0975² + 0.036²) = 0.151 * (0.02847 + 0.001296) = 0.00449 -->
-      <!-- Iyy = 1.81/12 * (3*0.0975² + 0.036²) = 0.151 * (0.02847 + 0.001296) = 0.00449 -->
-      <!-- Izz = 1.81/12 * (6*0.0975²) = 0.151 * 0.05693 = 0.00860 -->
-      <inertia ixx="0.00449" ixy="0.0" ixz="0.0"
-               iyy="0.00449" iyz="0.0"
-               izz="0.00860"/>
+      <mass value="${wheel_mass}"/>
+      <inertia ixx="${wheel_mass * (3*wheel_radius*wheel_radius + wheel_width*wheel_width) / 12}"
+               ixy="0.0" ixz="0.0"
+               iyy="${wheel_mass * wheel_radius*wheel_radius / 2}"
+               iyz="0.0"
+               izz="${wheel_mass * (3*wheel_radius*wheel_radius + wheel_width*wheel_width) / 12}"/>
     </inertial>
   </link>
-  <!-- Right wheel joint -->
-  <joint name="right_wheel_joint" type="continuous">
+  <!-- Left Wheel Joint -->
+  <joint name="left_wheel_joint" type="continuous">
     <parent link="base_link"/>
-    <child link="right_wheel"/>
-    <!-- Position: At (0, -23cm, 9.75cm) -->
-    <origin xyz="0.0 -0.23 0.0975" rpy="1.5707963 0 0"/>
-    <axis xyz="0 0 1"/>
+    <child link="left_wheel"/>
+    <origin xyz="0.0 ${wheel_separation/2} -${chassis_height/2}" rpy="0 0 0"/>
+    <axis xyz="0 1 0"/>
+    <dynamics damping="0.7" friction="1.0"/>
   </joint>
 </robot>
