Commit message: feat: Complete Phase 1 foundation with modular URDF and ros2_control integration

File: src/mower_description/urdf/mower.urdf.xacro (robot description, xacro)
@@ -18,8 +18,10 @@
   -->
   <!-- Include all component files -->
+  <xacro:include filename="$(find mower_description)/urdf/components/properties.xacro"/>
   <xacro:include filename="$(find mower_description)/urdf/components/materials.xacro"/>
   <xacro:include filename="$(find mower_description)/urdf/components/chassis.xacro"/>
   <xacro:include filename="$(find mower_description)/urdf/components/wheels.xacro"/>
   <xacro:include filename="$(find mower_description)/urdf/components/cutting_system.xacro"/>
+  <xacro:include filename="$(find mower_description)/urdf/components/sensors.xacro"/>
   <xacro:include filename="$(find mower_description)/urdf/components/ros2_control.xacro"/>
 </robot>

Commit message: feat(localization): replace dual-gps heading with ground truth and also changes to ekfs and navsat

File: src/mower_description/urdf/components/chassis.xacro (robot description, xacro)
@@ -9,13 +9,13 @@
   -->
   <!-- Root Link (dummy link without inertia for KDL compatibility) -->
-  <link name="base_footprint">
+  <!-- <link name="base_footprint"> -->
     <!-- No inertia on root link - KDL requirement -->
-  </link>
+  <!-- </link> -->
   <!-- Fixed joint connecting root to actual chassis -->
-  <joint name="base_footprint_joint" type="fixed">
-    <parent link="base_footprint"/>
-    <child link="base_link"/>
-    <origin xyz="0 0 ${wheel_radius}" rpy="0 0 0"/>
-  </joint>
+  <!-- <joint name="base_footprint_joint" type="fixed"> -->
+    <!-- <parent link="base_footprint"/> -->
+    <!-- <child link="base_link"/> -->
+    <!-- <origin xyz="0 0 ${wheel_radius}" rpy="0 0 0"/> -->
+  <!-- </joint> -->
   <!-- Base Link (main chassis) - now as child link with inertia -->
   <link name="base_link">

File: src/mower_description/urdf/components/properties.xacro (robot description, xacro)
@@ -36,12 +36,7 @@
   <xacro:property name="imu_y" value="0.0875" />
   <xacro:property name="imu_z" value="0.169" />
-  <!-- GPS sensor positions (dual GPS setup with 43cm baseline) -->
-  <!-- GPS Left sensor position -->
-  <xacro:property name="gps_left_x" value="0.0" />
-  <xacro:property name="gps_left_y" value="0.215" />
-  <xacro:property name="gps_left_z" value="0.253" />
-  <!-- GPS Right sensor position -->
-  <xacro:property name="gps_right_x" value="0.0" />
-  <xacro:property name="gps_right_y" value="-0.215" />
-  <xacro:property name="gps_right_z" value="0.253" />
+  <!-- GPS sensor position -->
+  <xacro:property name="gps_x" value="0.0" />
+  <xacro:property name="gps_y" value="0.215" />
+  <xacro:property name="gps_z" value="0.253" />
 </robot>

File: src/mower_description/urdf/components/sensors.xacro (robot description, xacro)
@@ -32,6 +32,6 @@
     <origin xyz="${imu_x} ${imu_y} ${imu_z - wheel_radius}" rpy="0 0 0"/>
   </joint>
-  <!-- GPS Left Sensor Link -->
-  <link name="gps_left_link">
+  <!-- GPS Sensor Link -->
+  <link name="gps_link">
     <visual>
       <geometry>
@@ -50,33 +50,9 @@
     </inertial>
   </link>
-  <!-- GPS Left Sensor Joint -->
-  <joint name="base_to_gps_left" type="fixed">
+  <!-- GPS Sensor Joint -->
+  <joint name="base_to_gps" type="fixed">
     <parent link="base_link"/>
-    <child link="gps_left_link"/>
-    <origin xyz="${gps_left_x} ${gps_left_y} ${gps_left_z - wheel_radius}" rpy="0 0 0"/>
-  </joint>
-  <!-- GPS Right Sensor Link -->
-  <link name="gps_right_link">
-    <visual>
-      <geometry>
-        <box size="0.03 0.03 0.04"/>
-      </geometry>
-      <material name="orange"/>
-    </visual>
-    <collision>
-      <geometry>
-        <box size="0.03 0.03 0.04"/>
-      </geometry>
-    </collision>
-    <inertial>
-      <mass value="0.01"/>
-      <inertia ixx="0.000001" ixy="0.0" ixz="0.0" iyy="0.000001" iyz="0.0" izz="0.000001"/>
-    </inertial>
-  </link>
-  <!-- GPS Right Sensor Joint -->
-  <joint name="base_to_gps_right" type="fixed">
-    <parent link="base_link"/>
-    <child link="gps_right_link"/>
-    <origin xyz="${gps_right_x} ${gps_right_y} ${gps_right_z - wheel_radius}" rpy="0 0 0"/>
+    <child link="gps_link"/>
+    <origin xyz="${gps_x} ${gps_y} ${gps_z - wheel_radius}" rpy="0 0 0"/>
   </joint>
   <!-- Gazebo IMU Sensor (native gz-sim format) -->
@@ -147,59 +123,21 @@
     </sensor>
   </gazebo>
-  <!-- Gazebo GPS Left Sensor (native gz-sim format) -->
-  <gazebo reference="gps_left_link">
-    <sensor name="gps_left_sensor" type="navsat">
+  <!-- Gazebo GPS Sensor (native gz-sim format) -->
+  <gazebo reference="gps_link">
+    <sensor name="gps_sensor" type="navsat">
       <always_on>1</always_on>
       <update_rate>20</update_rate>
       <visualize>true</visualize>
-      <topic>gps/left/fix</topic>
+      <topic>/gps/fix</topic>
       <navsat>
-        <position_sensing>
-          <horizontal>
-            <noise type="gaussian">
-              <mean>0.0</mean>
-              <stddev>0.01</stddev>
-              <bias_mean>0.0</bias_mean>
-              <bias_stddev>0.001</bias_stddev>
-            </noise>
-          </horizontal>
-          <vertical>
-            <noise type="gaussian">
-              <mean>0.0</mean>
-              <stddev>0.02</stddev>
-              <bias_mean>0.0</bias_mean>
-              <bias_stddev>0.002</bias_stddev>
-            </noise>
-          </vertical>
-        </position_sensing>
-      </navsat>
-    </sensor>
-  </gazebo>
-  <!-- Gazebo GPS Right Sensor (native gz-sim format) -->
-  <gazebo reference="gps_right_link">
-    <sensor name="gps_right_sensor" type="navsat">
-      <always_on>1</always_on>
-      <update_rate>20</update_rate>
-      <visualize>true</visualize>
-      <topic>gps/right/fix</topic>
-      <navsat>
-        <position_sensing>
-          <horizontal>
-            <noise type="gaussian">
-              <mean>0.0</mean>
-              <stddev>0.01</stddev>
-              <bias_mean>0.0</bias_mean>
-              <bias_stddev>0.001</bias_stddev>
-            </noise>
-          </horizontal>
-          <vertical>
-            <noise type="gaussian">
-              <mean>0.0</mean>
-              <stddev>0.02</stddev>
-              <bias_mean>0.0</bias_mean>
-              <bias_stddev>0.002</bias_stddev>
-            </noise>
-          </vertical>
-        </position_sensing>
+        <noise>
+          <type>gaussian</type>
+          <mean>0.0</mean>
+          <stddev>
+            <latitude>0.00001</latitude>
+            <longitude>0.00001</longitude>
+            <altitude>0.01</altitude>
+          </stddev>
+        </noise>
       </navsat>
     </sensor>

Commit message: feat(localization,bringup): wire ground_truth heading using gz model pose bridge; update node to geometry_msgs/Pose; single-GPS wiring

File: src/mower_description/urdf/components/chassis.xacro (robot description, xacro)
@@ -9,13 +9,13 @@
   -->
   <!-- Root Link (dummy link without inertia for KDL compatibility) -->
-  <!-- <link name="base_footprint"> -->
+  <link name="base_footprint">
     <!-- No inertia on root link - KDL requirement -->
-  <!-- </link> -->
+  </link>
   <!-- Fixed joint connecting root to actual chassis -->
-  <!-- <joint name="base_footprint_joint" type="fixed"> -->
-    <!-- <parent link="base_footprint"/> -->
-    <!-- <child link="base_link"/> -->
-    <!-- <origin xyz="0 0 ${wheel_radius}" rpy="0 0 0"/> -->
-  <!-- </joint> -->
+  <joint name="base_footprint_joint" type="fixed">
+    <parent link="base_footprint"/>
+    <child link="base_link"/>
+    <origin xyz="0 0 ${wheel_radius}" rpy="0 0 0"/>
+  </joint>
   <!-- Base Link (main chassis) - now as child link with inertia -->
   <link name="base_link">

File: src/mower_description/urdf/components/cutting_system.xacro (robot description, xacro)
@@ -99,5 +99,5 @@
     <parent link="base_link"/>
     <child link="reel_motor"/>
-    <origin xyz="0.125 0.11 0.04" rpy="0 0 0"/>
+    <origin xyz="0.125 -0.18 0.04" rpy="0 0 0"/>
   </joint>
 </robot>

File: src/mower_description/urdf/components/properties.xacro (robot description, xacro)
@@ -40,3 +40,4 @@
   <xacro:property name="gps_y" value="0.215" />
   <xacro:property name="gps_z" value="0.253" />
+  <xacro:property name="gps_yaw" value="1.5708" />
 </robot>

File: src/mower_description/urdf/components/sensors.xacro (robot description, xacro)
@@ -54,5 +54,5 @@
     <parent link="base_link"/>
     <child link="gps_link"/>
-    <origin xyz="${gps_x} ${gps_y} ${gps_z - wheel_radius}" rpy="0 0 0"/>
+    <origin xyz="${gps_x} ${gps_y} ${gps_z - wheel_radius}" rpy="0 0 ${gps_yaw}"/>
   </joint>
   <!-- Gazebo IMU Sensor (native gz-sim format) -->
