Commit message: Add dual GPS sensor configuration for Task 1.2

File: src/mower_description/urdf/components/properties.xacro (robot description, xacro)
@@ -36,7 +36,12 @@
   <xacro:property name="imu_y" value="0.0875" />
   <xacro:property name="imu_z" value="0.169" />
-  <!-- GPS sensor position -->
-  <xacro:property name="gps_x" value="0.0" />
-  <xacro:property name="gps_y" value="0.21415" />
-  <xacro:property name="gps_z" value="0.253" />
+  <!-- GPS sensor positions (dual GPS setup with 43cm baseline) -->
+  <!-- GPS Left sensor position -->
+  <xacro:property name="gps_left_x" value="0.0" />
+  <xacro:property name="gps_left_y" value="0.215" />
+  <xacro:property name="gps_left_z" value="0.253" />
+  <!-- GPS Right sensor position -->
+  <xacro:property name="gps_right_x" value="0.0" />
+  <xacro:property name="gps_right_y" value="-0.215" />
+  <xacro:property name="gps_right_z" value="0.253" />
 </robot>

File: src/mower_description/urdf/components/sensors.xacro (robot description, xacro)
@@ -32,6 +32,6 @@
     <origin xyz="${imu_x} ${imu_y} ${imu_z - wheel_radius}" rpy="0 0 0"/>
   </joint>
-  <!-- GPS Sensor Link -->
-  <link name="gps_link">
+  <!-- GPS Left Sensor Link -->
+  <link name="gps_left_link">
     <visual>
       <geometry>
@@ -50,9 +50,33 @@
     </inertial>
   </link>
-  <!-- GPS Sensor Joint -->
-  <joint name="base_to_gps" type="fixed">
+  <!-- GPS Left Sensor Joint -->
+  <joint name="base_to_gps_left" type="fixed">
     <parent link="base_link"/>
-    <child link="gps_link"/>
-    <origin xyz="${gps_x} ${gps_y} ${gps_z - wheel_radius}" rpy="0 0 0"/>
+    <child link="gps_left_link"/>
+    <origin xyz="${gps_left_x} ${gps_left_y} ${gps_left_z - wheel_radius}" rpy="0 0 0"/>
+  </joint>
+  <!-- GPS Right Sensor Link -->
+  <link name="gps_right_link">
+    <visual>
+      <geometry>
+        <box size="0.03 0.03 0.04"/>
+      </geometry>
+      <material name="orange"/>
+    </visual>
+    <collision>
+      <geometry>
+        <box size="0.03 0.03 0.04"/>
+      </geometry>
+    </collision>
+    <inertial>
+      <mass value="0.01"/>
+      <inertia ixx="0.000001" ixy="0.0" ixz="0.0" iyy="0.000001" iyz="0.0" izz="0.000001"/>
+    </inertial>
+  </link>
+  <!-- GPS Right Sensor Joint -->
+  <joint name="base_to_gps_right" type="fixed">
+    <parent link="base_link"/>
+    <child link="gps_right_link"/>
+    <origin xyz="${gps_right_x} ${gps_right_y} ${gps_right_z - wheel_radius}" rpy="0 0 0"/>
   </joint>
   <!-- Gazebo IMU Sensor (native gz-sim format) -->
@@ -64,4 +88,8 @@
       <topic>imu</topic>
       <imu>
+        <orientation_reference_frame>
+          <localization>ENU</localization>
+        </orientation_reference_frame>
+        <enable_orientation>true</enable_orientation>
         <angular_velocity>
           <x>
@@ -119,3 +147,61 @@
     </sensor>
   </gazebo>
+  <!-- Gazebo GPS Left Sensor (native gz-sim format) -->
+  <gazebo reference="gps_left_link">
+    <sensor name="gps_left_sensor" type="navsat">
+      <always_on>1</always_on>
+      <update_rate>20</update_rate>
+      <visualize>true</visualize>
+      <topic>gps/left/fix</topic>
+      <navsat>
+        <position_sensing>
+          <horizontal>
+            <noise type="gaussian">
+              <mean>0.0</mean>
+              <stddev>2.0</stddev>
+              <bias_mean>0.0</bias_mean>
+              <bias_stddev>0.1</bias_stddev>
+            </noise>
+          </horizontal>
+          <vertical>
+            <noise type="gaussian">
+              <mean>0.0</mean>
+              <stddev>4.0</stddev>
+              <bias_mean>0.0</bias_mean>
+              <bias_stddev>0.2</bias_stddev>
+            </noise>
+          </vertical>
+        </position_sensing>
+      </navsat>
+    </sensor>
+  </gazebo>
+  <!-- Gazebo GPS Right Sensor (native gz-sim format) -->
+  <gazebo reference="gps_right_link">
+    <sensor name="gps_right_sensor" type="navsat">
+      <always_on>1</always_on>
+      <update_rate>20</update_rate>
+      <visualize>true</visualize>
+      <topic>gps/right/fix</topic>
+      <navsat>
+        <position_sensing>
+          <horizontal>
+            <noise type="gaussian">
+              <mean>0.0</mean>
+              <stddev>2.0</stddev>
+              <bias_mean>0.0</bias_mean>
+              <bias_stddev>0.1</bias_stddev>
+            </noise>
+          </horizontal>
+          <vertical>
+            <noise type="gaussian">
+              <mean>0.0</mean>
+              <stddev>4.0</stddev>
+              <bias_mean>0.0</bias_mean>
+              <bias_stddev>0.2</bias_stddev>
+            </noise>
+          </vertical>
+        </position_sensing>
+      </navsat>
+    </sensor>
+  </gazebo>
 </robot>

Commit message: Phase 2: Sensors + Dual EKF (Simulation)
Merging Phase 2 after validation tests (Module 4 complete).

File: src/mower_description/urdf/components/properties.xacro (robot description, xacro)
@@ -38,5 +38,6 @@
   <!-- GPS sensor position -->
   <xacro:property name="gps_x" value="0.0" />
-  <xacro:property name="gps_y" value="0.21415" />
+  <xacro:property name="gps_y" value="0.215" />
   <xacro:property name="gps_z" value="0.253" />
+  <xacro:property name="gps_yaw" value="1.5708" />
 </robot>

File: src/mower_description/urdf/components/sensors.xacro (robot description, xacro)
@@ -54,5 +54,94 @@
     <parent link="base_link"/>
     <child link="gps_link"/>
-    <origin xyz="${gps_x} ${gps_y} ${gps_z - wheel_radius}" rpy="0 0 0"/>
+    <origin xyz="${gps_x} ${gps_y} ${gps_z - wheel_radius}" rpy="0 0 ${gps_yaw}"/>
   </joint>
+  <!-- Gazebo IMU Sensor (native gz-sim format) -->
+  <gazebo reference="imu_link">
+    <sensor name="imu_sensor" type="imu">
+      <always_on>1</always_on>
+      <update_rate>70</update_rate>
+      <visualize>true</visualize>
+      <topic>imu</topic>
+      <gz_frame_id>imu_link</gz_frame_id>
+      <imu>
+        <orientation_reference_frame>
+          <localization>ENU</localization>
+        </orientation_reference_frame>
+        <enable_orientation>true</enable_orientation>
+        <angular_velocity>
+          <x>
+            <noise type="gaussian">
+              <mean>0.0</mean>
+              <stddev>0.0005</stddev>
+              <bias_mean>0.0</bias_mean>
+              <bias_stddev>0.0001</bias_stddev>
+            </noise>
+          </x>
+          <y>
+            <noise type="gaussian">
+              <mean>0.0</mean>
+              <stddev>0.0005</stddev>
+              <bias_mean>0.0</bias_mean>
+              <bias_stddev>0.0001</bias_stddev>
+            </noise>
+          </y>
+          <z>
+            <noise type="gaussian">
+              <mean>0.0</mean>
+              <stddev>0.0005</stddev>
+              <bias_mean>0.0</bias_mean>
+              <bias_stddev>0.0001</bias_stddev>
+            </noise>
+          </z>
+        </angular_velocity>
+        <linear_acceleration>
+          <x>
+            <noise type="gaussian">
+              <mean>0.0</mean>
+              <stddev>0.005</stddev>
+              <bias_mean>0.0</bias_mean>
+              <bias_stddev>0.01</bias_stddev>
+            </noise>
+          </x>
+          <y>
+            <noise type="gaussian">
+              <mean>0.0</mean>
+              <stddev>0.005</stddev>
+              <bias_mean>0.0</bias_mean>
+              <bias_stddev>0.01</bias_stddev>
+            </noise>
+          </y>
+          <z>
+            <noise type="gaussian">
+              <mean>0.0</mean>
+              <stddev>0.005</stddev>
+              <bias_mean>0.0</bias_mean>
+              <bias_stddev>0.01</bias_stddev>
+            </noise>
+          </z>
+        </linear_acceleration>
+      </imu>
+    </sensor>
+  </gazebo>
+  <!-- Gazebo GPS Sensor (native gz-sim format) -->
+  <gazebo reference="gps_link">
+    <sensor name="gps_sensor" type="navsat">
+      <always_on>1</always_on>
+      <update_rate>20</update_rate>
+      <visualize>true</visualize>
+      <topic>/gps/fix</topic>
+      <gz_frame_id>gps_link</gz_frame_id>
+      <navsat>
+        <noise>
+          <type>gaussian</type>
+          <mean>0.0</mean>
+          <stddev>
+            <latitude>0.00000001</latitude>
+            <longitude>0.00000001</longitude>
+            <altitude>0.0000001</altitude>
+          </stddev>
+        </noise>
+      </navsat>
+    </sensor>
+  </gazebo>
 </robot>
